File: Power Supply.kicad_sch (KiCad schematic)
At the start: 17 parts, among them J1 Conn_01x02_Pin, J2 Conn_01x02_Pin, J3 Conn_01x03_Pin, J4 Conn_01x03_Pin, J5 Screw_Terminal_01x02, J6 Barrel_Jack, J7 Screw_Terminal_01x02, U1 LM7805_TO220, U2 LM317_TO-220

Commit message: just added a small text
Other:
- note added: "Just adding a text to test git"
Changed lines of the file:
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@@
+		)
+	)
+	(text "Just adding a text to test git"
+		(exclude_from_sim no)
+		(at 115.57 25.654 0)
+		(effects
+			(font
+				(size 2 2)
+			)
 		)
 	)

Commit message: Update Power Supply.kicad_sch
Other:
- note added: "Just adding a text to test github for learing github"
- note removed: "Just adding a text to test git"
Changed lines of the file:
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@@
 		)
 	)
-	(text "Just adding a text to test git"
+	(text "Just adding a text to test github for learing github"
 		(exclude_from_sim no)
 		(at 115.57 25.654 0)
